File: hardware/carrier/carrier.kicad_sch (KiCad schematic)
At the start: 80 parts, among them J1 PANEL+ / PANEL- (>=15 A, 4-6 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, J10 UART: 3V3 GND RX2(16) TX2(17), J11 5V / 5V SW / 3V3 / GND, J12 AUX + / - (>=15 A), J13 I2C: 3V3 GND SDA SCL, J14 ESP32 left row: EN,36,39,34,3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, J15 ESP32 right row: 23,22,1,3,21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, J2 BUCK IN + / -, J3 BUCK OUT + / - (set 5.0 V), J4 DS18B20: 3V3 / DATA / GND, J5 Optional 2nd probe, J6 Supercap 2.7 V 10 F (upper), J7 Supercap 2.7 V 10 F (lower), J8 microSD push-push with detect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, J9 Spare: 3V3 GND 32 33 36 26 27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, Q1 N-MOSFET >=60 V >=20 A Rds(on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, U1 DS3231SN (or RV-3028-C7, firm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, U2 INA180A3 (gain 100), U3 MCP1416 (or TC4427A class), U4 Load switch 5 V >=1 A, active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

Commit message: Carrier review 1: R2 4.7k (divider in ADC range), current-path and range notes on the schematic; firmware DIVIDER (6.1.1); BOM now tracked
Co-Authored-By: Claude Opus 5.5 <noreply@anthropic.com>
Claude-Session: https://claude.ai/code/session_01BMFMt5yCJVT3JQicJnUWqs
Parts:
- R2: value 5k6 1% -> 4k7 1%
Other:
- note added: "1. SUN-SENSOR LOOP: J1 -> D0 -> Q1 -> RSH1 -> GND Panel short-circuit current, ~1 ms every 10 s. Panel Isc 5.40 A (label), max ~6 A in cold strong sun. A vertical panel peaks near 1.8 A at noon. The panel cannot supply more than its Isc. 2. BOARD SUPPLY: PV+ -> F1 (2 A) -> D1 (3 A) -> buck -> +5V Under 0.3 A continuous. F1 and D1 are NOT in the measured current path: F1 sits after the Q1 node so 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"
- note added: "Current paths"
- note added: "ISENSE (GPIO 35): RSH1 5 mOhm x INA180A3 gain 100 = 0.5 V/A. Measured range 0-6 A (pulsed). 1.8 A -> 0.9 V; 5.4 A -> 2.7 V. Output clamps at the 3.3 V supply (~6.6 A): harmless. Gain 100 is deliberate: low vertical-panel currents stay well inside the ADC's range. Shunt dissipation 0.18 W only during each 1 ms pulse; 2 W rating is for pulse robustness. VDIV (GPIO 34): R1 100k / R2 4k7 = x 22.3 (R2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"
- note added: "Measurement ranges"

Commit message: Carrier review 2 (Copilot): R21 Q1 gate pull-down, D6 TVS footprint, AUX 3 A on v1, AP22804 verified, ESP32 module note
Co-Authored-By: Claude Opus 5.5 <noreply@anthropic.com>
Claude-Session: https://claude.ai/code/session_01BMFMt5yCJVT3JQicJnUWqs
Parts:
- added D6: DNP: SMCJ58A TVS (fit after bench test if needed), Diode_SMD:D_SMC, symbol Device:D_Zener
- added R21: 100k, Resistor_SMD:R_0603_1608Metric, symbol Device:R
- F4: value ATO blade holder, fuse NOT fitted (<=9 A) -> ATO blade holder, fuse NOT fitted (<=3 A on v1; 9 A only with D5 heatsink)
- Q1: value N-MOSFET >=60 V >=20 A Rds(on)<=20 mOhm @4.5 V -> N-MOSFET >=60 V (>=100 V if D6 fitted) >=20 A Rds(on)<=20 mOhm @4.5 V
Connections:
- net GATE: now also R21.1
- net GND: now also D6.2 (A)
- net PV+: now also D6.1 (K)
- net SHUNT_TOP: now also R21.2
Other:
- note added: "ESP32 module and Q1 gate (review 2)"
- note added: "The ESP32 is a complete ELEGOO dev board plugged into J14/J15. Its EN pull-up, reset and boot buttons, USB-serial converter and strapping resistors are on that board, not on the carrier. EN and GPIO 0, 1, 2, 3, 12, 15 are deliberately not brought out. GPIO 5 (strapping) is held high by R14. Q1 gate: U3 drives it when +5V exists; R21 (100k, gate-source) holds Q1 off before that, at dawn. D6 (TVS o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"
